File: usb.kicad_sch (KiCad schematic)
At the start: 10 parts

Commit message: complete mcu
Parts:
- gave numbers to parts that had none: 10
Changed lines of the file:
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@@
   (symbol (lib_id "power:GND") (at 247.65 115.57 0) (unit 1)
     (in_bom yes) (on_board yes) (fields_autoplaced)
-    (property "Reference" "#PWR?" (id 0) (at 247.65 121.92 0)
+    (property "Reference" "#PWR0155" (id 0) (at 247.65 121.92 0)
       (effects (font (size 1.27 1.27)) hide)
     )
@@
   (symbol (lib_id "power:GND") (at 158.75 93.98 90) (unit 1)
     (in_bom yes) (on_board yes) (fields_autoplaced)
-    (property "Reference" "#PWR?" (id 0) (at 165.1 93.98 0)
+    (property "Reference" "#PWR0153" (id 0) (at 165.1 93.98 0)
       (effects (font (size 1.27 1.27)) hide)
     )
@@
   (symbol (lib_id "power:GND") (at 212.09 115.57 0) (unit 1)
     (in_bom yes) (on_board yes) (fields_autoplaced)
-    (property "Reference" "#PWR?" (id 0) (at 212.09 121.92 0)
+    (property "Reference" "#PWR0154" (id 0) (at 212.09 121.92 0)
       (effects (font (size 1.27 1.27)) hide)
     )
@@
   (symbol (lib_id "Connector:USB_C_Receptacle_USB2.0") (at 128.27 102.87 0) (unit 1)
     (in_bom yes) (on_board yes) (fields_autoplaced)
-    (property "Reference" "J?" (id 0) (at 128.27 80.01 0))
+    (property "Reference" "J7" (id 0) (at 128.27 80.01 0))
     (property "Value" "USB_C_Receptacle_USB2.0" (id 1) (at 128.27 82.55 0))
     (property "Footprint" "" (id 2) (at 132.08 102.87 0)
@@
   (symbol (lib_id "Device:R") (at 151.13 92.71 90) (unit 1)
     (in_bom yes) (on_board yes)
-    (property "Reference" "R?" (id 0) (at 156.21 91.44 90))
+    (property "Reference" "R92" (id 0) (at 156.21 91.44 90))
     (property "Value" "5k1" (id 1) (at 151.13 92.71 90))
     (property "Footprint" "" (id 2) (at 151.13 94.488 90)
@@
   (symbol (lib_id "Device:R") (at 247.65 111.76 180) (unit 1)
     (in_bom yes) (on_board yes) (fields_autoplaced)
-    (property "Reference" "R?" (id 0) (at 250.19 110.4899 0)
+    (property "Reference" "R97" (id 0) (at 250.19 110.4899 0)
       (effects (font (size 1.27 1.27)) (justify right))
     )
@@
   (symbol (lib_id "Power_Protection:USBLC6-4SC6") (at 212.09 104.14 0) (unit 1)
     (in_bom yes) (on_board yes) (fields_autoplaced)
-    (property "Reference" "U?" (id 0) (at 214.8587 91.44 0)
+    (property "Reference" "U28" (id 0) (at 214.8587 91.44 0)
       (effects (font (size 1.27 1.27)) (justify left))
     )
@@
   (symbol (lib_id "Device:FerriteBead_Small") (at 191.77 87.63 90) (unit 1)
     (in_bom yes) (on_board yes) (fields_autoplaced)
-    (property "Reference" "FB?" (id 0) (at 191.7319 81.28 90))
+    (property "Reference" "FB12" (id 0) (at 191.7319 81.28 90))
     (property "Value" "1K@100MHz" (id 1) (at 191.7319 83.82 90))
     (property "Footprint" "" (id 2) (at 191.77 89.408 90)
@@
   (symbol (lib_id "Device:Filter_EMI_LL_1423") (at 175.26 104.14 0) (mirror x) (unit 1)
     (in_bom yes) (on_board yes) (fields_autoplaced)
-    (property "Reference" "FL?" (id 0) (at 174.879 96.52 0))
+    (property "Reference" "FL3" (id 0) (at 174.879 96.52 0))
     (property "Value" "90R@100MHz" (id 1) (at 174.879 99.06 0))
     (property "Footprint" "" (id 2) (at 175.26 97.79 0)
@@
   (symbol (lib_id "Device:R") (at 151.13 95.25 90) (unit 1)
     (in_bom yes) (on_board yes)
-    (property "Reference" "R?" (id 0) (at 156.21 93.98 90))
+    (property "Reference" "R93" (id 0) (at 156.21 93.98 90))
     (property "Value" "5k1" (id 1) (at 151.13 95.25 90))
     (property "Footprint" "" (id 2) (at 151.13 97.028 90)
@@
   (symbol (lib_id "Device:R") (at 232.41 87.63 90) (unit 1)
     (in_bom yes) (on_board yes)
-    (property "Reference" "R?" (id 0) (at 232.41 85.09 90))
+    (property "Reference" "R94" (id 0) (at 232.41 85.09 90))
     (property "Value" "5k1" (id 1) (at 232.41 90.17 90))
     (property "Footprint" "" (id 2) (at 232.41 89.408 90)
@@
   (symbol (lib_id "Device:R") (at 247.65 101.6 180) (unit 1)
     (in_bom yes) (on_board yes) (fields_autoplaced)
-    (property "Reference" "R?" (id 0) (at 250.19 100.3299 0)
+    (property "Reference" "R96" (id 0) (at 250.19 100.3299 0)
       (effects (font (size 1.27 1.27)) (justify right))
     )
@@
   (symbol (lib_id "Device:R") (at 247.65 91.44 180) (unit 1)
     (in_bom yes) (on_board yes) (fields_autoplaced)
-    (property "Reference" "R?" (id 0) (at 250.19 90.1699 0)
+    (property "Reference" "R95" (id 0) (at 250.19 90.1699 0)
       (effects (font (size 1.27 1.27)) (justify right))
     )
@@
   (symbol (lib_id "power:GND") (at 120.65 125.73 0) (unit 1)
     (in_bom yes) (on_board yes) (fields_autoplaced)
-    (property "Reference" "#PWR?" (id 0) (at 120.65 132.08 0)
-      (effects (font (size 1.27 1.27)) hide)
-    )
+    (property "Reference" "#PWR0152" (id 0) (at 120.65 132.08 0)
+      (effects (font (size 1.27 1.27)) hide)
+    )

Commit message: Complete BOM, FP assignment
Parts:
- FB12: footprint (none) -> Inductor_SMD:L_1210_3225Metric; MFR_PN (none) -> FBMH3225HM102NT; MFR_PN_ALT (none) -> FBMH3225HM102NTV
- FL3: footprint (none) -> Inductor_SMD:L_CommonModeChoke_Coilcraft_0603USB; MFR_PN (none) -> 0603USB-222MLC; MFR_PN_ALT (none) -> 0603USB-951MLC
- J7: footprint (none) -> Connector_USB:USB_C_Receptacle_HRO_TYPE-C-31-M-12; MFR_PN (none) -> TYPE-C-31-M-12; MFR_PN_ALT (none) -> USB4105-GF-A
- R92, R93, R94: footprint (none) -> Resistor_SMD:R_0603_1608Metric; MFR_PN (none) -> RMCF0603FT5K10; MFR_PN_ALT (none) -> CR0603-FX-5101ELF
- R95, R96, R97: footprint (none) -> Resistor_SMD:R_0603_1608Metric; MFR_PN (none) -> RNCP0603FTD10K0; MFR_PN_ALT (none) -> RMCF0603FT10K0
- U28: MFR_PN (none) -> USBLC6-4SC6Y; MFR_PN_ALT (none) -> USBLC6-4SC6
Changed lines of the file:
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@@
     (property "Reference" "J7" (id 0) (at 128.27 80.01 0))
     (property "Value" "USB_C_Receptacle_USB2.0" (id 1) (at 128.27 82.55 0))
-    (property "Footprint" "" (id 2) (at 132.08 102.87 0)
+    (property "Footprint" "Connector_USB:USB_C_Receptacle_HRO_TYPE-C-31-M-12" (id 2) (at 132.08 102.87 0)
       (effects (font (size 1.27 1.27)) hide)
     )
     (property "Datasheet" "https://www.usb.org/sites/default/files/documents/usb_type-c.zip" (id 3) (at 132.08 102.87 0)
+      (effects (font (size 1.27 1.27)) hide)
+    )
+    (property "MFR_PN" "TYPE-C-31-M-12" (id 4) (at 128.27 102.87 0)
+      (effects (font (size 1.27 1.27)) hide)
+    )
+    (property "MFR_PN_ALT" "USB4105-GF-A" (id 5) (at 128.27 102.87 0)
       (effects (font (size 1.27 1.27)) hide)
     )
@@
     (property "Reference" "R92" (id 0) (at 156.21 91.44 90))
     (property "Value" "5k1" (id 1) (at 151.13 92.71 90))
-    (property "Footprint" "" (id 2) (at 151.13 94.488 90)
+    (property "Footprint" "Resistor_SMD:R_0603_1608Metric" (id 2) (at 151.13 94.488 90)
       (effects (font (size 1.27 1.27)) hide)
     )
@@
       (effects (font (size 1.27 1.27)) hide)
     )
+    (property "MFR_PN" "RMCF0603FT5K10" (id 4) (at 151.13 92.71 0)
+      (effects (font (size 1.27 1.27)) hide)
+    )
+    (property "MFR_PN_ALT" "CR0603-FX-5101ELF" (id 5) (at 151.13 92.71 0)
+      (effects (font (size 1.27 1.27)) hide)
+    )
     (pin "1")
     (pin "2")
@@
       (effects (font (size 1.27 1.27)) (justify right))
     )
-    (property "Footprint" "" (id 2) (at 249.428 111.76 90)
+    (property "Footprint" "Resistor_SMD:R_0603_1608Metric" (id 2) (at 249.428 111.76 90)
       (effects (font (size 1.27 1.27)) hide)
     )
     (property "Datasheet" "~" (id 3) (at 247.65 111.76 0)
+      (effects (font (size 1.27 1.27)) hide)
+    )
+    (property "MFR_PN" "RNCP0603FTD10K0" (id 4) (at 247.65 111.76 0)
+      (effects (font (size 1.27 1.27)) hide)
+    )
+    (property "MFR_PN_ALT" "RMCF0603FT10K0" (id 5) (at 247.65 111.76 0)
       (effects (font (size 1.27 1.27)) hide)
     )
@@
     )
     (property "Datasheet" "https://www.st.com/resource/en/datasheet/usblc6-4.pdf" (id 3) (at 217.17 95.25 0)
+      (effects (font (size 1.27 1.27)) hide)
+    )
+    (property "MFR_PN" "USBLC6-4SC6Y" (id 4) (at 212.09 104.14 0)
+      (effects (font (size 1.27 1.27)) hide)
+    )
+    (property "MFR_PN_ALT" "USBLC6-4SC6" (id 5) (at 212.09 104.14 0)
       (effects (font (size 1.27 1.27)) hide)
     )
@@
     (property "Reference" "FB12" (id 0) (at 191.7319 81.28 90))
     (property "Value" "1K@100MHz" (id 1) (at 191.7319 83.82 90))
-    (property "Footprint" "" (id 2) (at 191.77 89.408 90)
+    (property "Footprint" "Inductor_SMD:L_1210_3225Metric" (id 2) (at 191.77 89.408 90)
       (effects (font (size 1.27 1.27)) hide)
     )
     (property "Datasheet" "~" (id 3) (at 191.77 87.63 0)
+      (effects (font (size 1.27 1.27)) hide)
+    )
+    (property "MFR_PN" "FBMH3225HM102NT" (id 4) (at 191.77 87.63 0)
+      (effects (font (size 1.27 1.27)) hide)
+    )
+    (property "MFR_PN_ALT" "FBMH3225HM102NTV" (id 5) (at 191.77 87.63 0)
       (effects (font (size 1.27 1.27)) hide)
     )
@@
     (property "Reference" "FL3" (id 0) (at 174.879 96.52 0))
     (property "Value" "90R@100MHz" (id 1) (at 174.879 99.06 0))
-    (property "Footprint" "" (id 2) (at 175.26 97.79 0)
+    (property "Footprint" "Inductor_SMD:L_CommonModeChoke_Coilcraft_0603USB" (id 2) (at 175.26 97.79 0)
       (effects (font (size 1.27 1.27)) hide)
     )
     (property "Datasheet" "~" (id 3) (at 175.26 105.156 90)
+      (effects (font (size 1.27 1.27)) hide)
+    )
+    (property "MFR_PN" "0603USB-222MLC" (id 4) (at 175.26 104.14 0)
+      (effects (font (size 1.27 1.27)) hide)
+    )
+    (property "MFR_PN_ALT" "0603USB-951MLC" (id 5) (at 175.26 104.14 0)
       (effects (font (size 1.27 1.27)) hide)
     )
@@
     (property "Reference" "R93" (id 0) (at 156.21 93.98 90))
     (property "Value" "5k1" (id 1) (at 151.13 95.25 90))
-    (property "Footprint" "" (id 2) (at 151.13 97.028 90)
+    (property "Footprint" "Resistor_SMD:R_0603_1608Metric" (id 2) (at 151.13 97.028 90)
       (effects (font (size 1.27 1.27)) hide)
     )
     (property "Datasheet" "~" (id 3) (at 151.13 95.25 0)
+      (effects (font (size 1.27 1.27)) hide)
+    )
+    (property "MFR_PN" "RMCF0603FT5K10" (id 4) (at 151.13 95.25 0)
+      (effects (font (size 1.27 1.27)) hide)
+    )
+    (property "MFR_PN_ALT" "CR0603-FX-5101ELF" (id 5) (at 151.13 95.25 0)
       (effects (font (size 1.27 1.27)) hide)
     )
@@
     (property "Reference" "R94" (id 0) (at 232.41 85.09 90))
     (property "Value" "5k1" (id 1) (at 232.41 90.17 90))
-    (property "Footprint" "" (id 2) (at 232.41 89.408 90)
+    (property "Footprint" "Resistor_SMD:R_0603_1608Metric" (id 2) (at 232.41 89.408 90)
       (effects (font (size 1.27 1.27)) hide)
     )
@@
       (effects (font (size 1.27 1.27)) hide)
     )
+    (property "MFR_PN" "RMCF0603FT5K10" (id 4) (at 232.41 87.63 0)
+      (effects (font (size 1.27 1.27)) hide)
+    )
+    (property "MFR_PN_ALT" "CR0603-FX-5101ELF" (id 5) (at 232.41 87.63 0)
+      (effects (font (size 1.27 1.27)) hide)
+    )
     (pin "1")
     (pin "2")
@@
       (effects (font (size 1.27 1.27)) (justify right))
     )
-    (property "Footprint" "" (id 2) (at 249.428 101.6 90)
+    (property "Footprint" "Resistor_SMD:R_0603_1608Metric" (id 2) (at 249.428 101.6 90)
       (effects (font (size 1.27 1.27)) hide)
     )
@@
       (effects (font (size 1.27 1.27)) hide)
     )
+    (property "MFR_PN" "RNCP0603FTD10K0" (id 4) (at 247.65 101.6 0)
+      (effects (font (size 1.27 1.27)) hide)
+    )
+    (property "MFR_PN_ALT" "RMCF0603FT10K0" (id 5) (at 247.65 101.6 0)
+      (effects (font (size 1.27 1.27)) hide)
+    )
     (pin "1")
     (pin "2")
@@
       (effects (font (size 1.27 1.27)) (justify right))
     )
-    (property "Footprint" "" (id 2) (at 249.428 91.44 90)
+    (property "Footprint" "Resistor_SMD:R_0603_1608Metric" (id 2) (at 249.428 91.44 90)
       (effects (font (size 1.27 1.27)) hide)
     )
@@
       (effects (font (size 1.27 1.27)) hide)
     )
+    (property "MFR_PN" "RNCP0603FTD10K0" (id 4) (at 247.65 91.44 0)
+      (effects (font (size 1.27 1.27)) hide)
+    )
+    (property "MFR_PN_ALT" "RMCF0603FT10K0" (id 5) (at 247.65 91.44 0)
+      (effects (font (size 1.27 1.27)) hide)
+    )

Commit message: sync
Parts:
- removed FL3: 90R@100MHz, Inductor_SMD:L_CommonModeChoke_Coilcraft_0603USB, symbol Device:Filter_EMI_LL_1423
- added FL3: 90R@100MHz, Inductor_SMD:L_CommonModeChoke_Coilcraft_0603USB, symbol kirdy:Filter_EMI_LL_1423
Connections:
- net USB_N: now also FL3.3
- net USB_P: now also FL3.2
- net at J7.A6 (D+), J7.B6 (D+): now also FL3.1
- net at J7.A7 (D-), J7.B7 (D-): now also FL3.4
Changed lines of the file:
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@@
     (pin "2")
-  )
-  (symbol (lib_id "Device:Filter_EMI_LL_1423") (at 175.26 104.14 0) (mirror x) (unit 1)
-    (in_bom yes) (on_board yes) (fields_autoplaced)
-    (property "Reference" "FL3" (id 0) (at 174.879 96.52 0))
-    (property "Value" "90R@100MHz" (id 1) (at 174.879 99.06 0))
-    (property "Footprint" "Inductor_SMD:L_CommonModeChoke_Coilcraft_0603USB" (id 2) (at 175.26 97.79 0)
-      (effects (font (size 1.27 1.27)) hide)
-    )
-    (property "Datasheet" "~" (id 3) (at 175.26 105.156 90)
-      (effects (font (size 1.27 1.27)) hide)
-    )
-    (property "MFR_PN" "0603USB-222MLC" (id 4) (at 175.26 104.14 0)
-      (effects (font (size 1.27 1.27)) hide)
-    )
-    (property "MFR_PN_ALT" "0603USB-951MLC" (id 5) (at 175.26 104.14 0)
-      (effects (font (size 1.27 1.27)) hide)
-    )
-    (pin "1")
-    (pin "2")
-    (pin "3")
-    (pin "4")
   )
   (symbol (lib_id "Device:R") (at 151.13 95.25 90) (unit 1)
@@
     (pin "2")
   )
+  (symbol (lib_id "kirdy:Filter_EMI_LL_1423") (at 175.26 104.14 0) (mirror x) (unit 1)
+    (in_bom yes) (on_board yes)
+    (property "Reference" "FL3" (id 0) (at 174.879 111.76 0))
+    (property "Value" "90R@100MHz" (id 1) (at 174.879 109.22 0))
+    (property "Footprint" "Inductor_SMD:L_CommonModeChoke_Coilcraft_0603USB" (id 2) (at 175.26 105.156 0)
+      (effects (font (size 1.27 1.27)) hide)
+    )
+    (property "Datasheet" "~" (id 3) (at 175.26 105.156 0)
+      (effects (font (size 1.27 1.27)) hide)
+    )
+    (property "MFR_PN" "0603USB-222MLC" (id 4) (at 175.26 104.14 0)
+      (effects (font (size 1.27 1.27)) hide)
+    )
+    (property "MFR_PN_ALT" "0603USB-951MLC" (id 5) (at 175.26 104.14 0)
+      (effects (font (size 1.27 1.27)) hide)
+    )
+    (pin "1")
+    (pin "2")
+    (pin "3")
+    (pin "4")
+  )
   (symbol (lib_id "power:GND") (at 120.65 125.73 0) (unit 1)

Commit message: some layout
Connections:
- net USB_N: now also FL3.2, U28.3 (I/O2); no longer FL3.3, U28.1 (I/O1)
- net USB_P: now also FL3.3, U28.1 (I/O1); no longer FL3.2, U28.3 (I/O2)
- net at J7.A6 (D+), J7.B6 (D+): now also FL3.4; no longer FL3.1
- net at J7.A7 (D-), J7.B7 (D-): now also FL3.1; no longer FL3.4
Other:
- moved on the sheet: R94
Changed lines of the file:
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@@
   (junction (at 143.51 106.68) (diameter 0) (color 0 0 0 0)
   )
-  (junction (at 212.09 87.63) (diameter 0) (color 0 0 0 0)
+  (junction (at 232.41 87.63) (diameter 0) (color 0 0 0 0)
   )
   (junction (at 247.65 106.68) (diameter 0) (color 0 0 0 0)
@@
     (stroke (width 0) (type default) (color 0 0 0 0))
   )
+  (wire (pts (xy 212.09 91.44) (xy 212.09 93.98))
+    (stroke (width 0) (type default) (color 0 0 0 0))
+  )
   (wire (pts (xy 143.51 87.63) (xy 189.23 87.63))
     (stroke (width 0) (type default) (color 0 0 0 0))
@@
     (stroke (width 0) (type default) (color 0 0 0 0))
   )
+  (wire (pts (xy 209.55 91.44) (xy 212.09 91.44))
+    (stroke (width 0) (type default) (color 0 0 0 0))
+  )
   (wire (pts (xy 247.65 105.41) (xy 247.65 106.68))
     (stroke (width 0) (type default) (color 0 0 0 0))
@@
     (stroke (width 0) (type default) (color 0 0 0 0))
   )
+  (wire (pts (xy 247.65 106.68) (xy 247.65 107.95))
+    (stroke (width 0) (type default) (color 0 0 0 0))
+  )
+  (wire (pts (xy 158.75 93.98) (xy 158.75 92.71))
+    (stroke (width 0) (type default) (color 0 0 0 0))
+  )
+  (wire (pts (xy 180.34 101.6) (xy 185.42 101.6))
+    (stroke (width 0) (type default) (color 0 0 0 0))
+  )
+  (wire (pts (xy 247.65 95.25) (xy 247.65 97.79))
+    (stroke (width 0) (type default) (color 0 0 0 0))
+  )
   (wire (pts (xy 212.09 115.57) (xy 212.09 114.3))
     (stroke (width 0) (type default) (color 0 0 0 0))
   )
-  (wire (pts (xy 247.65 106.68) (xy 247.65 107.95))
-    (stroke (width 0) (type default) (color 0 0 0 0))
-  )
-  (wire (pts (xy 158.75 93.98) (xy 158.75 92.71))
-    (stroke (width 0) (type default) (color 0 0 0 0))
-  )
-  (wire (pts (xy 180.34 101.6) (xy 185.42 101.6))
-    (stroke (width 0) (type default) (color 0 0 0 0))
-  )
-  (wire (pts (xy 247.65 95.25) (xy 247.65 97.79))
-    (stroke (width 0) (type default) (color 0 0 0 0))
-  )
   (wire (pts (xy 143.51 101.6) (xy 143.51 102.87))
     (stroke (width 0) (type default) (color 0 0 0 0))
   )
+  (wire (pts (xy 232.41 87.63) (xy 236.22 87.63))
+    (stroke (width 0) (type default) (color 0 0 0 0))
+  )
   (wire (pts (xy 143.51 105.41) (xy 143.51 106.68))
     (stroke (width 0) (type default) (color 0 0 0 0))
   )
-  (wire (pts (xy 236.22 87.63) (xy 247.65 87.63))
+  (wire (pts (xy 243.84 87.63) (xy 247.65 87.63))
     (stroke (width 0) (type default) (color 0 0 0 0))
   )
@@
     (stroke (width 0) (type default) (color 0 0 0 0))
   )
-  (wire (pts (xy 212.09 87.63) (xy 212.09 93.98))
-    (stroke (width 0) (type default) (color 0 0 0 0))
-  )
   (wire (pts (xy 185.42 101.6) (xy 201.93 101.6))
     (stroke (width 0) (type default) (color 0 0 0 0))
   )
-  (wire (pts (xy 194.31 87.63) (xy 212.09 87.63))
-    (stroke (width 0) (type default) (color 0 0 0 0))
-  )
   (wire (pts (xy 143.51 101.6) (xy 170.18 101.6))
     (stroke (width 0) (type default) (color 0 0 0 0))
@@
     (stroke (width 0) (type default) (color 0 0 0 0))
   )
+  (wire (pts (xy 232.41 87.63) (xy 232.41 115.57))
+    (stroke (width 0) (type default) (color 0 0 0 0))
+  )
   (wire (pts (xy 143.51 95.25) (xy 147.32 95.25))
     (stroke (width 0) (type default) (color 0 0 0 0))
@@
     (stroke (width 0) (type default) (color 0 0 0 0))
   )
-  (wire (pts (xy 212.09 87.63) (xy 228.6 87.63))
+  (wire (pts (xy 194.31 87.63) (xy 232.41 87.63))
+    (stroke (width 0) (type default) (color 0 0 0 0))
+  )
+  (wire (pts (xy 232.41 115.57) (xy 212.09 115.57))
     (stroke (width 0) (type default) (color 0 0 0 0))
   )
@@
     (pin "1")
   )
-  (symbol (lib_id "power:GND") (at 212.09 115.57 0) (unit 1)
-    (in_bom yes) (on_board yes) (fields_autoplaced)
-    (property "Reference" "#PWR0154" (id 0) (at 212.09 121.92 0)
-      (effects (font (size 1.27 1.27)) hide)
-    )
-    (property "Value" "GND" (id 1) (at 212.09 120.65 0))
-    (property "Footprint" "" (id 2) (at 212.09 115.57 0)
-      (effects (font (size 1.27 1.27)) hide)
-    )
-    (property "Datasheet" "" (id 3) (at 212.09 115.57 0)
+  (symbol (lib_id "power:GND") (at 209.55 91.44 270) (unit 1)
+    (in_bom yes) (on_board yes) (fields_autoplaced)
+    (property "Reference" "#PWR0154" (id 0) (at 203.2 91.44 0)
+      (effects (font (size 1.27 1.27)) hide)
+    )
+    (property "Value" "GND" (id 1) (at 205.74 91.4399 90)
+      (effects (font (size 1.27 1.27)) (justify right))
+    )
+    (property "Footprint" "" (id 2) (at 209.55 91.44 0)
+      (effects (font (size 1.27 1.27)) hide)
+    )
+    (property "Datasheet" "" (id 3) (at 209.55 91.44 0)
       (effects (font (size 1.27 1.27)) hide)
     )
@@
     (pin "2")
   )
-  (symbol (lib_id "Power_Protection:USBLC6-4SC6") (at 212.09 104.14 0) (unit 1)
+  (symbol (lib_id "Power_Protection:USBLC6-4SC6") (at 212.09 104.14 0) (mirror x) (unit 1)
     (in_bom yes) (on_board yes) (fields_autoplaced)
     (property "Reference" "U28" (id 0) (at 214.8587 91.44 0)
@@
       (effects (font (size 1.27 1.27)) (justify left))
     )
-    (property "Footprint" "Package_TO_SOT_SMD:SOT-23-6" (id 2) (at 212.09 116.84 0)
-      (effects (font (size 1.27 1.27)) hide)
-    )
-    (property "Datasheet" "https://www.st.com/resource/en/datasheet/usblc6-4.pdf" (id 3) (at 217.17 95.25 0)
+    (property "Footprint" "Package_TO_SOT_SMD:SOT-23-6" (id 2) (at 212.09 91.44 0)
+      (effects (font (size 1.27 1.27)) hide)
+    )
+    (property "Datasheet" "https://www.st.com/resource/en/datasheet/usblc6-4.pdf" (id 3) (at 217.17 113.03 0)
       (effects (font (size 1.27 1.27)) hide)
     )
@@
     (pin "2")
   )
-  (symbol (lib_id "Device:R") (at 232.41 87.63 90) (unit 1)
+  (symbol (lib_id "Device:R") (at 240.03 87.63 90) (unit 1)
     (in_bom yes) (on_board yes)
-    (property "Reference" "R94" (id 0) (at 232.41 85.09 90))
-    (property "Value" "5k1" (id 1) (at 232.41 90.17 90))
-    (property "Footprint" "Resistor_SMD:R_0603_1608Metric" (id 2) (at 232.41 89.408 90)
-      (effects (font (size 1.27 1.27)) hide)
-    )
-    (property "Datasheet" "~" (id 3) (at 232.41 87.63 0)
-      (effects (font (size 1.27 1.27)) hide)
-    )
-    (property "MFR_PN" "RMCF0603FT5K10" (id 4) (at 232.41 87.63 0)
-      (effects (font (size 1.27 1.27)) hide)
-    )
-    (property "MFR_PN_ALT" "CR0603-FX-5101ELF" (id 5) (at 232.41 87.63 0)
+    (property "Reference" "R94" (id 0) (at 240.03 85.09 90))
+    (property "Value" "5k1" (id 1) (at 240.03 90.17 90))
+    (property "Footprint" "Resistor_SMD:R_0603_1608Metric" (id 2) (at 240.03 89.408 90)
+      (effects (font (size 1.27 1.27)) hide)
+    )
+    (property "Datasheet" "~" (id 3) (at 240.03 87.63 0)
+      (effects (font (size 1.27 1.27)) hide)
+    )
+    (property "MFR_PN" "RMCF0603FT5K10" (id 4) (at 240.03 87.63 0)
+      (effects (font (size 1.27 1.27)) hide)
+    )
+    (property "MFR_PN_ALT" "CR0603-FX-5101ELF" (id 5) (at 240.03 87.63 0)
       (effects (font (size 1.27 1.27)) hide)
     )
@@
     (pin "2")
   )
-  (symbol (lib_id "kirdy:Filter_EMI_LL_1423") (at 175.26 104.14 0) (mirror x) (unit 1)
+  (symbol (lib_id "kirdy:Filter_EMI_LL_1423") (at 175.26 104.14 0) (unit 1)
     (in_bom yes) (on_board yes)
-    (property "Reference" "FL3" (id 0) (at 174.879 111.76 0))
-    (property "Value" "90R@100MHz" (id 1) (at 174.879 109.22 0))
-    (property "Footprint" "Inductor_SMD:L_CommonModeChoke_Coilcraft_0603USB" (id 2) (at 175.26 105.156 0)
-      (effects (font (size 1.27 1.27)) hide)
-    )
-    (property "Datasheet" "~" (id 3) (at 175.26 105.156 0)
-      (effects (font (size 1.27 1.27)) hide)
-    )
+    (property "Reference" "FL3" (id 0) (at 174.879 96.52 0))
+    (property "Value" "90R@100MHz" (id 1) (at 174.879 99.06 0))
+    (property "Footprint" "Inductor_SMD:L_CommonModeChoke_Coilcraft_0603USB" (id 2) (at 175.26 103.124 0)
+      (effects (font (size 1.27 1.27)) hide)
+    )
+    (property "Datasheet" "~" (id 3) (at 175.26 103.124 0)
+      (effects (font (size 1.27 1.27)) hide)
+    )
