File: kirdy.kicad_pcb (KiCad board)
At the start: 4 copper layers, 160 x 100 mm, 387 parts, among them J1 MOD_IN, J2 Conn_01x10, J3 Conn_01x10, J4 Conn_02x05_Odd_Even, J5 Barrel_Jack, J6 RJ45_Abracon_ARJP11A-MASA-B-A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, J7 USB_C_Receptacle_USB2.0, J8 Conn_02x05_Odd_Even, J9 Conn_02x05_Odd_Even, K1 DIP12-1C90-51L, Q1 SQJA70EP-T1, Q2 BSS138, Q3 BSS138, Q4 BC857, Q5 AOSP21321, Q6 BC857, Q7 BSS138, SW1 SW_DIP_x03, U1 LTC6655BHLS8-4.096, U10 LT3081xDF, U11 LT3042xMSE, U12 LT3045xMSE, U13 LT3045xMSE, U14 LT3042xMSE, U15 LT3094xMSE, U16 LT3042xMSE, U17 AD5680, U18 AD7172-2, U19 RS8552, U2 MAX5719xSD, U20 MAX1968xUI, U21 ACPL-217-500E, U22 TPS54620, U24 PM1202, U25 AMS1117-3.3, U26 LAN8742A, U27 USBLC6-4SC6, U28 USBLC6-4SC6, U3 ADA4898-1YRDZ, U4 ADA4898-1YRDZ, U5 LM358, U6 ADA4898-1YRDZ, U7 STM32F407VGTx, U8 STM809SWX6F, U9 LTC3261, Y1 8MHz, Y2 25MHz

Commit message: fix eth
Routing:
- removed copper zone on B.Cu, net +15V
- removed copper zone on B.Cu, net +9VA
- removed copper zone on B.Cu, net /Ehternet/ETH_SHIELD
Changed lines of the file:
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@@
       (pts
-        (xy 140.462 18.542)
         (xy 140.462 18.542)
         (xy 140.462 22.733)
@@
       )
     )
-  )
-  (zone (net 85) (net_name "/Ehternet/ETH_SHIELD") (layer "B.Cu") (hatch edge 0.508)
-    (priority 6)
-    (connect_pads yes (clearance 0.254))
-    (min_thickness 0.254) (filled_areas_thickness no)
-    (fill yes (thermal_gap 0.508) (thermal_bridge_width 0.508) (smoothing fillet) (radius 0.5))
-    (polygon
-      (pts
-        (xy 16.764 73.025)
-        (xy 8.001 73.025)
-        (xy 8.001 53.467)
-        (xy 16.764 53.467)
-      )
-    )
-  )
-  (zone (net 9) (net_name "+15V") (layer "B.Cu") (hatch edge 0.508)
-    (priority 6)
-    (connect_pads yes (clearance 0.254))
-    (min_thickness 0.254) (filled_areas_thickness no)
-    (fill yes (thermal_gap 0.508) (thermal_bridge_width 0.508) (smoothing fillet) (radius 0.5))
-    (polygon
-      (pts
-        (xy 136.652 37.084)
-        (xy 107.696 37.084)
-        (xy 107.696 52.324)
-        (xy 102.616 52.324)
-        (xy 102.87 32.258)
-        (xy 133.35 32.258)
-        (xy 133.35 22.86)
-        (xy 128.778 22.86)
-        (xy 128.778 13.716)
-        (xy 136.652 13.716)
-      )
-    )
-  )
-  (zone (net 7) (net_name "+9VA") (layer "B.Cu") (hatch edge 0.508)
-    (priority 6)
-    (connect_pads yes (clearance 0.254))
-    (min_thickness 0.254) (filled_areas_thickness no)
-    (fill yes (thermal_gap 0.508) (thermal_bridge_width 0.508) (smoothing fillet) (radius 0.5))
-    (polygon
-      (pts
-        (xy 128.27 23.622)
-        (xy 132.588 23.622)
-        (xy 132.588 31.496)
-        (xy 102.108 31.496)
-        (xy 102.108 38.862)
-        (xy 61.214 38.862)
-        (xy 61.214 24.892)
-        (xy 119.888 24.892)
-        (xy 119.888 9.652)
-        (xy 128.27 9.652)
-      )
-    )

Commit message: placement v2
Parts:
- removed R18: 300, Resistor_SMD:R_0603_1608Metric
- added R107: 100, Resistor_SMD:R_0603_1608Metric, F.Cu at (24.4, 49.6)
- added R108: 100, Resistor_SMD:R_0603_1608Metric, F.Cu at (24.4, 45.1)
- added R109: 100, Resistor_SMD:R_0603_1608Metric, F.Cu at (24.3, 42.7)
- added R110: 100, Resistor_SMD:R_0603_1608Metric, F.Cu at (28.8, 42.7)
- moved Q2 42.4 mm to (23.1, 89.9), turned to 0 degrees
- moved R56 42.0 mm to (23.6, 87.2), turned to 0 degrees
- moved R57 33.0 mm to (22.6, 74.6), turned to 90 degrees
- moved J2 29.1 mm to (65.7, 28.6)
- moved C156 28.8 mm to (87.8, 64.0), turned to 90 degrees
- moved U21 27.7 mm to (30.4, 89.2), turned to 0 degrees
- moved L9 26.6 mm to (91.1, 63.7), turned to 0 degrees
- moved C154 26.3 mm to (83.5, 64.0)
- moved C153 26.3 mm to (85.7, 64.0)
- moved R62 26.2 mm to (39.9, 90.6)
- moved R16 26.0 mm to (64.0, 60.2)
- moved Q3 25.9 mm to (42.5, 90.2)
- moved C18 25.3 mm to (66.3, 60.2)
- moved C26 25.2 mm to (67.9, 60.2)
- moved C30 24.6 mm to (49.6, 47.8)
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Connections:
- net +1V8 renamed Net-(C35-Pad1)
- R85 pad 1: /Ehternet/PHY_TD_P -> /Ehternet/PHY_RD_N
- R86 pad 1: /Ehternet/PHY_TD_N -> /Ehternet/PHY_RD_P
- R87 pad 1: /Ehternet/PHY_RD_P -> /Ehternet/PHY_TD_N
- R88 pad 1: /Ehternet/PHY_RD_N -> /Ehternet/PHY_TD_P
- U27 pad 4: /Ehternet/PHY_TD_P -> /Ehternet/PHY_TD_N
- U27 pad 6: /Ehternet/PHY_TD_N -> /Ehternet/PHY_TD_P
Routing:
- removed copper zone on F.Cu, net +12V
- removed copper zone on F.Cu, net +15V
- removed copper zone on F.Cu, net +3.3VA
- removed copper zone on F.Cu, net +3V3
- removed copper zone on F.Cu, net +5V
- removed copper zone on In2.Cu, net +5V
- removed copper zone on F.Cu, net +5VA
- removed copper zone on In2.Cu, net +5VA
- removed copper zone on F.Cu, net +8V
- removed copper zone on F.Cu, net +9VA
- removed copper zone on F.Cu, net -9V
- removed copper zone on F.Cu, net /Ehternet/ETH_SHIELD
- removed copper zone on F.Cu, net /Ehternet/POE_VC-
- removed copper zone on F.Cu, net /driveStage/LD-
- removed copper zone on F.Cu, net /thermostat/TEC+
- removed copper zone on F.Cu, net /thermostat/TEC-
- removed copper zone on F.Cu, net IN
- removed copper zone on F.Cu, net Net-(C135-Pad2)
- removed copper zone on F.Cu, net Net-(C136-Pad2)
- removed copper zone on F.Cu, net Net-(C145-Pad1)
- removed copper zone on F.Cu, net Net-(C145-Pad2)
- removed copper zone on F.Cu, net Net-(C158-Pad1)
- removed copper zone on F.Cu, net Net-(C35-Pad1)
- removed copper zone on F.Cu, net Net-(C37-Pad2)
- removed copper zone on F.Cu, net Net-(C40-Pad1)
- removed copper zone on F.Cu, net Net-(C42-Pad2)
- removed copper zone on F.Cu, net Net-(C43-Pad2)
- removed copper zone on F.Cu, net Net-(C50-Pad1)
- removed copper zone on F.Cu, net Net-(C52-Pad1)
- removed copper zone on F.Cu, net Net-(C53-Pad1)
- removed copper zone on F.Cu, net Net-(C54-Pad1)
- removed copper zone on F.Cu, net Net-(C55-Pad1)
- removed copper zone on F.Cu, net Net-(L2-Pad1)
- removed copper zone on F.Cu, net Net-(L3-Pad1)
- removed copper zone on F.Cu, net Net-(Q1-Pad1)
- removed copper zone on F.Cu, net Net-(R45-Pad1)
Other:
- board text removed: "2.5mA/V"
- board text removed: "250uA/V"
- board text removed: "25mA/V"

Commit message: update palcement
Parts:
- FL1: value 5A -> 2x1m
- moved J4 4.72 mm to (67.7, 35.9)
- moved C35 4.00 mm to (95.3, 46.3)
- moved C36 4.00 mm to (88.5, 47.0)
- moved C40 4.00 mm to (80.9, 57.1)
- moved C178 4.00 mm to (89.7, 51.7)
- moved C179 4.00 mm to (89.5, 49.7)
- moved C180 4.00 mm to (90.8, 57.1)
- moved C32 4.00 mm to (85.8, 57.1)
- moved C33 4.00 mm to (86.0, 49.5)
- moved C34 4.00 mm to (86.0, 51.5)
- moved C37 4.00 mm to (96.9, 50.4)
- moved C38 4.00 mm to (101.0, 46.4)
- moved C39 4.00 mm to (93.5, 46.5)
- moved C41 4.00 mm to (98.7, 50.2)
- moved C42 4.00 mm to (104.2, 46.4)
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Other:
- board text added: "V0.2 Precision laser driver"
- board text removed: "V0.1 Precision laser driver"

Commit message: some layout
Parts:
- moved J3 23.7 mm to (42.0, 24.0), turned to 90 degrees
- moved R91 22.9 mm to (14.1, 75.6), turned to 0 degrees
- moved C171 20.5 mm to (14.7, 73.5)
- moved C145 13.7 mm to (39.9, 74.0)
- moved R110 7.79 mm to (21.1, 43.5)
- moved R97 6.79 mm to (14.3, 52.1)
- moved C90 5.96 mm to (78.6, 30.9), turned to 180 degrees
- moved C76 5.72 mm to (78.8, 32.7), turned to 180 degrees
- moved R88 4.77 mm to (22.6, 43.5)
- moved R23 4.28 mm to (82.5, 29.5), turned to 0 degrees
- moved R104 3.99 mm to (144.6, 47.3)
- moved D12 3.99 mm to (151.5, 46.4)
- moved Q7 3.99 mm to (148.3, 46.4)
- moved R103 3.99 mm to (144.6, 45.6)
- moved C83 3.80 mm to (78.6, 34.5), turned to 180 degrees
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Connections:
- FL3 pad 2: /MCU/USB_DP -> /MCU/USB_DN
- FL3 pad 3: /MCU/USB_DN -> /MCU/USB_DP
- J7 pad A6: Net-(FL3-Pad1) -> Net-(FL3-Pad4)
- J7 pad A7: Net-(FL3-Pad4) -> Net-(FL3-Pad1)
- J7 pad B6: Net-(FL3-Pad1) -> Net-(FL3-Pad4)
- J7 pad B7: Net-(FL3-Pad4) -> Net-(FL3-Pad1)
- U28 pad 1: /MCU/USB_DN -> /MCU/USB_DP
- U28 pad 3: /MCU/USB_DP -> /MCU/USB_DN
- U7 pad 35: /MCU/TEC_ISEN -> /MCU/TEC_VSEN
- U7 pad 36: /MCU/TEC_VSEN -> /MCU/TEC_ISEN
Routing:
- net /MCU/LD_EN: track 0.00 -> 141.9 mm
- net Net-(D1-Pad2): track 0.00 -> 122.6 mm
- net /MCU/TADC_CLK: track 0.00 -> 104.9 mm, vias 0 -> 2
- net /MCU/TADC_MISO: track 0.00 -> 103.3 mm, vias 0 -> 2
- net /MCU/TADC_CS: track 0.00 -> 101.9 mm, vias 0 -> 2
- net /MCU/~{LD_SHORT}: track 0.00 -> 101.5 mm, vias 0 -> 2
- net /MCU/TADC_SYNC: track 0.00 -> 101.3 mm, vias 0 -> 2
- net /MCU/PD_MON: track 0.00 -> 100.4 mm, vias 0 -> 2
- net /MCU/TADC_MOSI: track 0.00 -> 99.6 mm, vias 0 -> 2
- net /MCU/TEC_VSEN: track 0.00 -> 93.6 mm, vias 0 -> 2
- net /MCU/TDAC_MOSI: track 0.00 -> 90.4 mm, vias 0 -> 2
- net /MCU/TDAC_CLK: track 0.00 -> 88.9 mm, vias 0 -> 2
- net /MCU/TDAC_SYNC: track 0.00 -> 87.2 mm, vias 0 -> 2
- net /MCU/TEC_VREF: track 0.00 -> 86.9 mm, vias 0 -> 2
- net /MCU/TEC_SHDN: track 0.00 -> 80.6 mm, vias 0 -> 2
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