File: dsupply.kicad_sch (KiCad schematic)
At the start: 66 parts, among them J8 Barrel_Jack, Q3 BC857, Q4 AOSP21321, Q5 AOSP21321, Q6 BC857, Q7 BC857, Q8 AOSP21321, Q9 BC857, U22 PM1202, U23 TPS54620, U24 AMS1117-3.3

Commit message: sch, pcb: Correct MFR/PN and optimize BOM
Parts:
- C184: MFR_PN CL10B104KB8NNW -> CL10B105KA8NNNC; MFR_PN_ALT CL10B104KB8NNNL -> CGA3E1X7R1E105K080AC
Changed lines of the file:
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@@
   (symbol (lib_id "power:GND") (at 196.215 46.99 0) (mirror y) (unit 1)
     (in_bom yes) (on_board yes) (dnp no) (fields_autoplaced)
-    (property "Reference" "#PWR0153" (at 196.215 53.34 0)
+    (property "Reference" "#PWR0154" (at 196.215 53.34 0)
       (effects (font (size 1.27 1.27)) hide)
     )
@@
       (project "kirdy"
         (path "/88da1dd8-9274-4b55-84fb-90006c9b6e8f/b6f53a06-e1b9-4c20-8fc0-ae2d1ce0191d"
-          (reference "#PWR0153") (unit 1)
+          (reference "#PWR0154") (unit 1)
         )
       )
@@
   (symbol (lib_id "power:GND") (at 274.32 111.125 0) (unit 1)
     (in_bom yes) (on_board yes) (dnp no) (fields_autoplaced)
-    (property "Reference" "#PWR0160" (at 274.32 117.475 0)
+    (property "Reference" "#PWR0161" (at 274.32 117.475 0)
       (effects (font (size 1.27 1.27)) hide)
     )
@@
       (project "kirdy"
         (path "/88da1dd8-9274-4b55-84fb-90006c9b6e8f/b6f53a06-e1b9-4c20-8fc0-ae2d1ce0191d"
-          (reference "#PWR0160") (unit 1)
+          (reference "#PWR0161") (unit 1)
         )
       )
@@
   (symbol (lib_id "power:+12V") (at 378.46 76.2 0) (unit 1)
     (in_bom yes) (on_board yes) (dnp no) (fields_autoplaced)
-    (property "Reference" "#PWR0166" (at 378.46 80.01 0)
+    (property "Reference" "#PWR0167" (at 378.46 80.01 0)
       (effects (font (size 1.27 1.27)) hide)
     )
@@
       (project "kirdy"
         (path "/88da1dd8-9274-4b55-84fb-90006c9b6e8f/b6f53a06-e1b9-4c20-8fc0-ae2d1ce0191d"
-          (reference "#PWR0166") (unit 1)
+          (reference "#PWR0167") (unit 1)
         )
       )
@@
   (symbol (lib_id "power:GND") (at 241.935 111.125 0) (unit 1)
     (in_bom yes) (on_board yes) (dnp no) (fields_autoplaced)
-    (property "Reference" "#PWR0156" (at 241.935 117.475 0)
+    (property "Reference" "#PWR0157" (at 241.935 117.475 0)
       (effects (font (size 1.27 1.27)) hide)
     )
@@
       (project "kirdy"
         (path "/88da1dd8-9274-4b55-84fb-90006c9b6e8f/b6f53a06-e1b9-4c20-8fc0-ae2d1ce0191d"
-          (reference "#PWR0156") (unit 1)
+          (reference "#PWR0157") (unit 1)
         )
       )
@@
   (symbol (lib_id "power:GND") (at 73.66 170.18 0) (unit 1)
     (in_bom yes) (on_board yes) (dnp no) (fields_autoplaced)
-    (property "Reference" "#PWR0151" (at 73.66 176.53 0)
+    (property "Reference" "#PWR0152" (at 73.66 176.53 0)
       (effects (font (size 1.27 1.27)) hide)
     )
@@
       (project "kirdy"
         (path "/88da1dd8-9274-4b55-84fb-90006c9b6e8f/b6f53a06-e1b9-4c20-8fc0-ae2d1ce0191d"
-          (reference "#PWR0151") (unit 1)
+          (reference "#PWR0152") (unit 1)
         )
       )
@@
   (symbol (lib_id "power:+5V") (at 246.38 157.48 0) (unit 1)
     (in_bom yes) (on_board yes) (dnp no) (fields_autoplaced)
-    (property "Reference" "#PWR0158" (at 246.38 161.29 0)
+    (property "Reference" "#PWR0159" (at 246.38 161.29 0)
       (effects (font (size 1.27 1.27)) hide)
     )
@@
       (project "kirdy"
         (path "/88da1dd8-9274-4b55-84fb-90006c9b6e8f/b6f53a06-e1b9-4c20-8fc0-ae2d1ce0191d"
-          (reference "#PWR0158") (unit 1)
+          (reference "#PWR0159") (unit 1)
         )
       )
@@
   (symbol (lib_id "power:GND") (at 327.025 111.125 0) (unit 1)
     (in_bom yes) (on_board yes) (dnp no) (fields_autoplaced)
-    (property "Reference" "#PWR0163" (at 327.025 117.475 0)
+    (property "Reference" "#PWR0164" (at 327.025 117.475 0)
       (effects (font (size 1.27 1.27)) hide)
     )
@@
       (project "kirdy"
         (path "/88da1dd8-9274-4b55-84fb-90006c9b6e8f/b6f53a06-e1b9-4c20-8fc0-ae2d1ce0191d"
-          (reference "#PWR0163") (unit 1)
+          (reference "#PWR0164") (unit 1)
         )
       )
@@
   (symbol (lib_id "power:GND") (at 179.07 86.36 0) (unit 1)
     (in_bom yes) (on_board yes) (dnp no) (fields_autoplaced)
-    (property "Reference" "#PWR0152" (at 179.07 92.71 0)
+    (property "Reference" "#PWR0153" (at 179.07 92.71 0)
       (effects (font (size 1.27 1.27)) hide)
     )
@@
       (project "kirdy"
         (path "/88da1dd8-9274-4b55-84fb-90006c9b6e8f/b6f53a06-e1b9-4c20-8fc0-ae2d1ce0191d"
-          (reference "#PWR0152") (unit 1)
+          (reference "#PWR0153") (unit 1)
         )
       )
@@
   (symbol (lib_id "power:GND") (at 378.46 86.36 0) (unit 1)
     (in_bom yes) (on_board yes) (dnp no) (fields_autoplaced)
-    (property "Reference" "#PWR0167" (at 378.46 92.71 0)
+    (property "Reference" "#PWR0168" (at 378.46 92.71 0)
       (effects (font (size 1.27 1.27)) hide)
     )
@@
       (project "kirdy"
         (path "/88da1dd8-9274-4b55-84fb-90006c9b6e8f/b6f53a06-e1b9-4c20-8fc0-ae2d1ce0191d"
-          (reference "#PWR0167") (unit 1)
+          (reference "#PWR0168") (unit 1)
         )
       )
@@
   (symbol (lib_id "power:GND") (at 214.63 91.44 0) (unit 1)
     (in_bom yes) (on_board yes) (dnp no) (fields_autoplaced)
-    (property "Reference" "#PWR0154" (at 214.63 97.79 0)
+    (property "Reference" "#PWR0155" (at 214.63 97.79 0)
       (effects (font (size 1.27 1.27)) hide)
     )
@@
       (project "kirdy"
         (path "/88da1dd8-9274-4b55-84fb-90006c9b6e8f/b6f53a06-e1b9-4c20-8fc0-ae2d1ce0191d"
-          (reference "#PWR0154") (unit 1)
+          (reference "#PWR0155") (unit 1)
         )
       )
@@
   (symbol (lib_id "power:GND") (at 294.64 111.125 0) (unit 1)
     (in_bom yes) (on_board yes) (dnp no) (fields_autoplaced)
-    (property "Reference" "#PWR0162" (at 294.64 117.475 0)
+    (property "Reference" "#PWR0163" (at 294.64 117.475 0)
       (effects (font (size 1.27 1.27)) hide)
     )
@@
       (project "kirdy"
         (path "/88da1dd8-9274-4b55-84fb-90006c9b6e8f/b6f53a06-e1b9-4c20-8fc0-ae2d1ce0191d"
-          (reference "#PWR0162") (unit 1)
+          (reference "#PWR0163") (unit 1)
         )
       )
@@
   (symbol (lib_id "power:GND") (at 251.46 182.88 0) (unit 1)
     (in_bom yes) (on_board yes) (dnp no) (fields_autoplaced)
-    (property "Reference" "#PWR0159" (at 251.46 189.23 0)
+    (property "Reference" "#PWR0160" (at 251.46 189.23 0)
       (effects (font (size 1.27 1.27)) hide)
     )
@@
       (project "kirdy"
         (path "/88da1dd8-9274-4b55-84fb-90006c9b6e8f/b6f53a06-e1b9-4c20-8fc0-ae2d1ce0191d"
-          (reference "#PWR0159") (unit 1)
+          (reference "#PWR0160") (unit 1)
         )
       )
@@
   (symbol (lib_id "power:GND") (at 246.38 52.07 0) (mirror y) (unit 1)
     (in_bom yes) (on_board yes) (dnp no)
-    (property "Reference" "#PWR0157" (at 246.38 58.42 0)
+    (property "Reference" "#PWR0158" (at 246.38 58.42 0)
       (effects (font (size 1.27 1.27)) hide)
     )
@@
       (project "kirdy"
         (path "/88da1dd8-9274-4b55-84fb-90006c9b6e8f/b6f53a06-e1b9-4c20-8fc0-ae2d1ce0191d"
-          (reference "#PWR0157") (unit 1)
+          (reference "#PWR0158") (unit 1)
         )
       )
@@
       (effects (font (size 1.27 1.27)) hide)
     )
-    (property "MFR_PN" "CL10B104KB8NNW" (at 232.41 36.83 0)
-      (effects (font (size 1.27 1.27)) hide)
-    )
-    (property "MFR_PN_ALT" "CL10B104KB8NNNL" (at 232.41 36.83 0)
+    (property "MFR_PN" "CL10B105KA8NNNC" (at 232.41 36.83 0)
+      (effects (font (size 1.27 1.27)) hide)
+    )
+    (property "MFR_PN_ALT" "CGA3E1X7R1E105K080AC" (at 232.41 36.83 0)
       (effects (font (size 1.27 1.27)) hide)
     )
@@
   (symbol (lib_id "power:GND") (at 336.55 165.1 0) (unit 1)
     (in_bom yes) (on_board yes) (dnp no) (fields_autoplaced)
-    (property "Reference" "#PWR0164" (at 336.55 171.45 0)
+    (property "Reference" "#PWR0165" (at 336.55 171.45 0)
       (effects (font (size 1.27 1.27)) hide)
     )
@@
       (project "kirdy"
         (path "/88da1dd8-9274-4b55-84fb-90006c9b6e8f/b6f53a06-e1b9-4c20-8fc0-ae2d1ce0191d"
-          (reference "#PWR0164") (unit 1)
+          (reference "#PWR0165") (unit 1)
         )
       )
@@
   (symbol (lib_id "power:+12V") (at 53.34 149.86 90) (unit 1)
     (in_bom yes) (on_board yes) (dnp no) (fields_autoplaced)
-    (property "Reference" "#PWR0150" (at 57.15 149.86 0)
+    (property "Reference" "#PWR0151" (at 57.15 149.86 0)
       (effects (font (size 1.27 1.27)) hide)
     )
@@
       (project "kirdy"
         (path "/88da1dd8-9274-4b55-84fb-90006c9b6e8f/b6f53a06-e1b9-4c20-8fc0-ae2d1ce0191d"
-          (reference "#PWR0150") (unit 1)
+          (reference "#PWR0151") (unit 1)
         )
       )
@@
   (symbol (lib_id "power:GND") (at 232.41 52.07 0) (mirror y) (unit 1)
     (in_bom yes) (on_board yes) (dnp no)
-    (property "Reference" "#PWR0155" (at 232.41 58.42 0)
+    (property "Reference" "#PWR0156" (at 232.41 58.42 0)
       (effects (font (size 1.27 1.27)) hide)
     )
@@
       (project "kirdy"
         (path "/88da1dd8-9274-4b55-84fb-90006c9b6e8f/b6f53a06-e1b9-4c20-8fc0-ae2d1ce0191d"
-          (reference "#PWR0155") (unit 1)
+          (reference "#PWR0156") (unit 1)
         )
       )
@@
   (symbol (lib_id "power:+3V3") (at 364.49 157.48 0) (unit 1)
     (in_bom yes) (on_board yes) (dnp no) (fields_autoplaced)
-    (property "Reference" "#PWR0165" (at 364.49 161.29 0)
+    (property "Reference" "#PWR0166" (at 364.49 161.29 0)
       (effects (font (size 1.27 1.27)) hide)
     )
@@
       (project "kirdy"
         (path "/88da1dd8-9274-4b55-84fb-90006c9b6e8f/b6f53a06-e1b9-4c20-8fc0-ae2d1ce0191d"
-          (reference "#PWR0165") (unit 1)
+          (reference "#PWR0166") (unit 1)
         )
       )
@@
   (symbol (lib_id "power:GND") (at 289.56 182.88 0) (unit 1)
     (in_bom yes) (on_board yes) (dnp no) (fields_autoplaced)
-    (property "Reference" "#PWR0161" (at 289.56 189.23 0)
+    (property "Reference" "#PWR0162" (at 289.56 189.23 0)
       (effects (font (size 1.27 1.27)) hide)
     )
@@
       (project "kirdy"
         (path "/88da1dd8-9274-4b55-84fb-90006c9b6e8f/b6f53a06-e1b9-4c20-8fc0-ae2d1ce0191d"
-          (reference "#PWR0161") (unit 1)
-        )
-      )
+          (reference "#PWR0162") (unit 1)
+        )
+      )
